File: hw_balanceo/bat_balancing/bat_balancing.sch (KiCad schematic (older format))
At the start: 36 parts, among them J4 Conn_01x07, J5 NTC, J6 NTC, J7 Conn_REG50, U1 bq76pl536

Commit message: First charger sch version.
TODO:
	+ Imput Snubber

	+ Select Q & N power MOS

	+ Calc L & C

	+ Tempr Sens
Parts:
- U1: symbol Battery_Management:bq76pl536 -> bat_balancing-rescue:bq76pl536-Battery_Management
- U?: symbol MCU_Microchip_ATmega:ATmega328P-AU -> bat_balancing-rescue:ATmega328P-AU-MCU_Microchip_ATmega
Changed lines of the file:
@@
 EESchema Schematic File Version 4
-LIBS:bat_balancing-cache
-EELAYER 26 0
+EELAYER 30 0
 EELAYER END
 $Descr A4 11693 8268
@@
 	6900 5450 6900 5350
 $Comp
-L Battery_Management:bq76pl536 U1
+L bat_balancing-rescue:bq76pl536-Battery_Management U1
 U 1 1 5C1DB3BA
 P 5650 4800
@@
 	3550 4850 4450 4850
 $Comp
-L MCU_Microchip_ATmega:ATmega328P-AU U?
+L bat_balancing-rescue:ATmega328P-AU-MCU_Microchip_ATmega U?
 U 1 1 5CA2BA08
 P 1750 2200
