File: hw_balanceo/bat_charging/bat_charging.sch (KiCad schematic (older format))
At the start: 56 parts

Commit message: Avances del esquematico:
            + Imput Snubber DONE!

            + Select Q & N power MOS DONE!

            + Calc L & C DONE!

TODO:
            + Tempr Sens
Parts:
- removed C?: 0.1a1uF, symbol Device:C
- removed C?: 0.1uF, symbol Device:C
- removed C?: 10uF, symbol Device:C
- removed D?: D, symbol Device:D
- removed J?: Conn_Coaxial_Power, symbol Connector:Conn_Coaxial_Power
- removed Q?: Q_PMOS_DGS, symbol Device:Q_PMOS_DGS
- removed R?: 4R7a30R, symbol Device:R
- removed R?: 100K, symbol Device:R
- removed R?: 1K, symbol Device:R
- added C12: 10uF, Capacitors_SMD:CP_Elec_6.3x7.7, symbol Device:CP
- added C6: 1uF, Capacitors_SMD:C_0805_HandSoldering, symbol Device:CP
- added J1: Vcc In, Connectors_Molex:Molex_KK-41791-02_02x3.96mm_Straight, symbol Connector_Generic:Conn_01x02
- added NT1: GND-TIE, Oddities:NetTie-I_Connected_SMD, symbol Device:Net-Tie_2
- added TP1: GND_BAT, Keystone_5016:KEYSTONE_5016, symbol Connector:TestPoint
- added TP2: GNDA, Keystone_5016:KEYSTONE_5016, symbol Connector:TestPoint
- added TP3: VREF, Keystone_5016:KEYSTONE_5016, symbol Connector:TestPoint
- added TP4: VBUS, Keystone_5016:KEYSTONE_5016, symbol Connector:TestPoint
- added TP5: VCC, Keystone_5016:KEYSTONE_5016, symbol Connector:TestPoint
- added TP6: CH_BAT, Keystone_5016:KEYSTONE_5016, symbol Connector:TestPoint
- C1: renamed from C?; value 2.2uF -> 2.7nF; footprint (none) -> Capacitors_SMD:C_0805_HandSoldering
- C10, C11, C2, C3, C4, C5, C7, C8, C9: renamed from C?; footprint (none) -> Capacitors_SMD:C_0805_HandSoldering
- C13, C14: renamed from C?; value C -> 10uF; footprint (none) -> Capacitors_SMD:CP_Elec_6.3x7.7; symbol Device:C -> Device:CP
- D1: renamed from D?; value D -> N4007; footprint (none) -> Diodes_THT:D_A-405_P7.62mm_Horizontal
- D2, D3, D4, D5: renamed from D?; footprint (none) -> LEDs:LED_0603_HandSoldering
- D6: renamed from D?; value D_Schottky -> RB541SM-40FHT2R; footprint (none) -> Diodes_SMD:D_SOD-523
- L1: renamed from L?; value L -> 6.8uH; footprint (none) -> BOURNS_SRP6030VA:SRP6030VA-6R8M
- Q1, Q2: renamed from Q?; value Q_PMOS_DGS -> Q_PMOS_GDS; footprint (none) -> TO_SOT_Packages_SMD:TO-252-2_Rectifier; symbol Device:Q_PMOS_DGS -> Device:Q_PMOS_GDS
- Q3, Q4: renamed from Q?; value Q_NMOS_DGS -> FDD86580-F085; footprint (none) -> TO_SOT_Packages_SMD:TO-252-2_Rectifier; symbol Device:Q_NMOS_DGS -> Device:Q_NMOS_GDS
- R1, R2, R6: renamed from R?; value 10K -> 10K*; footprint (none) -> Resistors_SMD:R_0805_HandSoldering
- R10, R11, R13, R9: renamed from R?; footprint (none) -> Resistors_SMD:R_0805_HandSoldering
- R12: renamed from R?; value 0R010⁯ -> 0R010⁯ 1W 0.5%; footprint (none) -> Resistors_SMD:R_1206_HandSoldering
- R14, R15, R16: renamed from R?; value 420R -> 470R; footprint (none) -> Resistors_SMD:R_0805_HandSoldering
- R19: renamed from R?; value 0R020 -> 0R020 1W 0.5%; footprint (none) -> Resistors_SMD:R_1206_HandSoldering
- R20: renamed from R?; value 1K -> 1K 1/8W 1%; footprint (none) -> Resistors_SMD:R_0805_HandSoldering
- R21: renamed from R?; value 560K -> 560K 1/10W 0.5%; footprint (none) -> Resistors_SMD:R_0805_HandSoldering
- R22: renamed from R?; value 51K -> 51K 1/8W 0.5%; footprint (none) -> Resistors_SMD:R_0805_HandSoldering
- R3: renamed from R?; value 37K -> 37K*; footprint (none) -> Resistors_SMD:R_0805_HandSoldering
- R4: renamed from R?; value 8K2 -> 8K2*; footprint (none) -> Resistors_SMD:R_0805_HandSoldering
- R5: renamed from R?; value 6K8 -> 6K8*; footprint (none) -> Resistors_SMD:R_0805_HandSoldering
- R7: renamed from R?; value 2R -> 6R2 1/4W 1%; footprint (none) -> Resistors_SMD:R_1206_HandSoldering
- R8: renamed from R?; value 10k -> 10k 1/8W 5%; footprint (none) -> Resistors_SMD:R_0805_HandSoldering
- SW1: renamed from SW?; value Reset CE -> Reset; footprint (none) -> Buttons_Switches_THT:SW_TH_Tactile_Omron_B3F-10xx
- SW2: renamed from SW?; value SW_DIP_x02 -> Select CE; footprint (none) -> Buttons_Switches_THT:SW_DIP_x2_W7.62mm_Piano
- U1: renamed from U?; footprint RGE24_2P45X2P45 -> lib:BQ24618RGET
Connections:
- net labels added: CH_BAT, CH_CE, CH_GNDA, CH_GND_BAT, CH_PG, CH_STAT1, CH_STAT2, EPAD, GND_BAT, VBUS
- net labels removed: +3.3V, GNDPWR, SYSTEM, VBAT, Vad+, uCE
- wire segments 197 -> 190
- no-connect marks 0 -> 1
Other:
- note added: "* 1 ON , 2 OFF: Stand Alone\n* 1 OFF , 2 ON : u Controlled"
- note added: "* 1/8W 0.5%"
- note added: "* Charge: CC-CV 0.5C (max) 4.20V, 100mA cut-off at 25°C"
- note added: "* Fast-charge safety timer range: Tcharge = 5hs / Cttc(C9) = 0.056uF *"
- note added: "* I (pre-charge) = V2set/(100*Rse)\n* I (fast charge) = V1set/(20*Rse)\n* Icset = max I imput = 5A"
- note added: "* Vref max load 35mA!! (Actual = 15,7mA)\n"
- note added: "*!BATDRV (o) should manage the battery to system gate, but the\n problem is it is referenced to ACN. ANC-6 < Vbatdrv < ACN"
- note added: "+VBATT = 2.1*[1+(R20+R21)/R22]"
- note added: "I & V Charging Set Points"
- note added: "Imput"
- note added: "Output"
- note added: "Reset & CE Source Selector"
- note added: "Status LEDs & Signals"
- note removed: "* Charge: CC-CV 0.5C (max) 4.20V, 100mA cut-off at 25°C\n* Fast-charge safety timer range: Tcharge = 5hs / Cttc =0.056uF * \n*"
- moved on the sheet: C1, C10, C11, C2, C3, C4, C5, C7, C8, C9, D1, D2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
