File: current_sensor_ina226.sch (KiCad schematic (older format))
At the start: 6 parts, among them U3 INA226

Commit message: Changes overlapping names of pins between bq76 and ina226
Connections:
- net ALERT renamed ALERT_INA226
Changed lines of the file:
@@
 $Descr A4 11693 8268
 encoding utf-8
-Sheet 5 5
+Sheet 4 5
 Title ""
 Date ""
@@
 SCL
 Text HLabel 7100 4200 2    50   Output ~ 0
-ALERT
+ALERT_INA226
 $Comp
 L Device:R R35
