File: current_sensor_ina226.sch (KiCad schematic (older format))
At the start: 6 parts, among them U3 INA226

Commit message: Dletes hw_balanceo folder
Parts:
- renumbered C37 to C1, R35 to R1, R36 to R2, R37 to R3, R38 to R4, U3 to U1
Changed lines of the file:
@@
 $EndDescr
 $Comp
-L Analog_ADC:INA226 U3
+L Analog_ADC:INA226 U1
 U 1 1 5FE92189
 P 5400 3900
-F 0 "U3" H 5400 4000 50  0000 C CNN
+F 0 "U1" H 5400 4000 50  0000 C CNN
 F 1 "INA226" H 5400 3900 50  0000 C CNN
 F 2 "Package_SO:VSSOP-10_3x3mm_P0.5mm" H 6200 3450 50  0001 C CNN
@@
 $EndComp
 $Comp
-L power:+3V3 #PWR0136
+L power:+3V3 #PWR010
 U 1 1 5FE94A7C
 P 5400 3400
-F 0 "#PWR0136" H 5400 3250 50  0001 C CNN
+F 0 "#PWR010" H 5400 3250 50  0001 C CNN
 F 1 "+3V3" H 5415 3573 50  0000 C CNN
 F 2 "" H 5400 3400 50  0001 C CNN
@@
 $EndComp
 $Comp
-L power:+3V3 #PWR0137
+L power:+3V3 #PWR014
 U 1 1 5FE96F31
 P 7750 3750
-F 0 "#PWR0137" H 7750 3600 50  0001 C CNN
+F 0 "#PWR014" H 7750 3600 50  0001 C CNN
 F 1 "+3V3" H 7765 3923 50  0000 C CNN
 F 2 "" H 7750 3750 50  0001 C CNN
@@
 $EndComp
 $Comp
-L Device:C C37
+L Device:C C1
 U 1 1 5FE97303
 P 7750 4000
-F 0 "C37" H 7865 4046 50  0000 L CNN
+F 0 "C1" H 7865 4046 50  0000 L CNN
 F 1 "0.1uF" H 7865 3955 50  0000 L CNN
 F 2 "Capacitor_SMD:C_0805_2012Metric_Pad1.18x1.45mm_HandSolder" H 7788 3850 50  0001 C CNN
@@
 	7750 3750 7750 3850
 $Comp
-L power:GND #PWR0138
+L power:GND #PWR015
 U 1 1 5FE97A9F
 P 7750 4250
-F 0 "#PWR0138" H 7750 4000 50  0001 C CNN
+F 0 "#PWR015" H 7750 4000 50  0001 C CNN
 F 1 "GND" H 7755 4077 50  0000 C CNN
 F 2 "" H 7750 4250 50  0001 C CNN
@@
 	7750 4150 7750 4250
 $Comp
-L power:GND #PWR0139
+L power:GND #PWR012
 U 1 1 5FE98538
 P 5900 3650
-F 0 "#PWR0139" H 5900 3400 50  0001 C CNN
+F 0 "#PWR012" H 5900 3400 50  0001 C CNN
 F 1 "GND" V 5905 3522 50  0000 R CNN
 F 2 "" H 5900 3650 50  0001 C CNN
@@
 	5850 3650 5850 3700
 $Comp
-L Device:R R36
+L Device:R R2
 U 1 1 5FE98DFC
 P 6300 3650
-F 0 "R36" H 6370 3696 50  0000 L CNN
+F 0 "R2" H 6370 3696 50  0000 L CNN
 F 1 "10K" H 6370 3605 50  0000 L CNN
 F 2 "Resistor_SMD:R_0805_2012Metric_Pad1.20x1.40mm_HandSolder" V 6230 3650 50  0001 C CNN
@@
 $EndComp
 $Comp
-L Device:R R37
+L Device:R R3
 U 1 1 5FE98FC7
 P 6600 3650
-F 0 "R37" H 6670 3696 50  0000 L CNN
+F 0 "R3" H 6670 3696 50  0000 L CNN
 F 1 "10K" H 6670 3605 50  0000 L CNN
 F 2 "Resistor_SMD:R_0805_2012Metric_Pad1.20x1.40mm_HandSolder" V 6530 3650 50  0001 C CNN
@@
 $EndComp
 $Comp
-L Device:R R38
+L Device:R R4
 U 1 1 5FE99104
 P 6900 3650
-F 0 "R38" H 6970 3696 50  0000 L CNN
+F 0 "R4" H 6970 3696 50  0000 L CNN
 F 1 "10K" H 6970 3605 50  0000 L CNN
 F 2 "Resistor_SMD:R_0805_2012Metric_Pad1.20x1.40mm_HandSolder" V 6830 3650 50  0001 C CNN
@@
 $EndComp
 $Comp
-L power:+3V3 #PWR0140
+L power:+3V3 #PWR013
 U 1 1 5FE99B82
 P 6600 3400
-F 0 "#PWR0140" H 6600 3250 50  0001 C CNN
+F 0 "#PWR013" H 6600 3250 50  0001 C CNN
 F 1 "+3V3" H 6615 3573 50  0000 C CNN
 F 2 "" H 6600 3400 50  0001 C CNN
@@
 	6900 4200 6900 3800
 $Comp
-L power:GND #PWR0141
+L power:GND #PWR011
 U 1 1 5FE9AFA5
 P 5400 4450
-F 0 "#PWR0141" H 5400 4200 50  0001 C CNN
+F 0 "#PWR011" H 5400 4200 50  0001 C CNN
 F 1 "GND" H 5405 4277 50  0000 C CNN
 F 2 "" H 5400 4450 50  0001 C CNN
@@
 ALERT_INA226
 $Comp
-L Device:R R35
+L Device:R R1
 U 1 1 5FE9DD8B
 P 4200 4050
-F 0 "R35" H 4270 4096 50  0000 L CNN
+F 0 "R1" H 4270 4096 50  0000 L CNN
 F 1 "2.5mOhm 1W 1%" H 4270 4005 50  0000 L CNN
 F 2 "Resistor_SMD:R_2512_6332Metric_Pad1.40x3.35mm_HandSolder" V 4130 4050 50  0001 C CNN

Commit message: Final version pcb
Parts:
- renumbered U1 to U9
Changed lines of the file:
@@
 $Descr A4 11693 8268
 encoding utf-8
-Sheet 2 8
+Sheet 2 9
 Title ""
 Date ""
@@
 $EndDescr
 $Comp
-L Analog_ADC:INA226 U1
+L Analog_ADC:INA226 U9
 U 1 1 5FE92189
 P 5400 3900
-F 0 "U1" H 5400 4000 50  0000 C CNN
+F 0 "U9" H 5400 4000 50  0000 C CNN
 F 1 "INA226" H 5400 3900 50  0000 C CNN
 F 2 "Package_SO:VSSOP-10_3x3mm_P0.5mm" H 6200 3450 50  0001 C CNN
