File: bat_switch.sch (KiCad schematic (older format))
At the start: 8 parts, among them Q11 BC848, Q12 BC848, Q13 IRF9310PbF, U5 FERD2045SB-TR

Commit message: Adds final pcb
Parts:
- U5: footprint Package_TO_SOT_SMD:TO-263-3_TabPin2 -> Package_TO_SOT_SMD:TO-252-2
Changed lines of the file:
@@
 U 1 1 6024EE1E
 P 6250 4500
-F 0 "U5" V 7250 3650 60  0000 L CNN
-F 1 "FERD2045SB-TR" V 7350 3300 60  0000 L CNN
-F 2 "Package_TO_SOT_SMD:TO-263-3_TabPin2" H 7050 4740 60  0001 C CNN
+F 0 "U5" V 7103 4072 60  0000 R CNN
+F 1 "FERD2045SB-TR" V 6997 4072 60  0000 R CNN
+F 2 "Package_TO_SOT_SMD:TO-252-2" H 7050 4740 60  0001 C CNN
 F 3 "https://ar.mouser.com/datasheet/2/389/ferd2045s-1849465.pdf" V 7156 4728 60  0001 L CNN
 	1    6250 4500
