File: bat_switch.sch (KiCad schematic (older format))
At the start: 8 parts, among them Q11 BC848, Q12 BC848, Q13 IRF9310PbF, U5 FERD2045SB-TR

Commit message: Edited sch page settings & printed schematic pdf
Parts:
- Q13: symbol Transistor_FET:IRF9310PbF -> bms_hardware-rescue:IRF9310PbF-Transistor_FET
- U5: symbol 2021-02-09_22-26-07:FERD2045SB-TR -> bms_hardware-rescue:FERD2045SB-TR-2021-02-09_22-26-07
Connections:
- net D: now also U5.3 (K); no longer U5.2 (K)
- net GND: now also U5.2 (A); no longer U5.3 (A)
Changed lines of the file:
@@
 encoding utf-8
 Sheet 7 9
-Title ""
+Title "Battery Managment System (MBS)"
 Date ""
 Rev "A"
-Comp ""
+Comp "Ceccarelli Federico, Moya Martin,  Santos Lucio"
 Comment1 ""
-Comment2 ""
-Comment3 ""
-Comment4 ""
+Comment2 "Universidad Nacional de Rosario (UNR)"
+Comment3 "Facultad de Ciencias Exactas, Ingeniería y Agrimensura"
+Comment4 "Proyecto Final - Ingeniería Electrónica"
 $EndDescr
 $Comp
@@
 	5800 4500 6150 4500
 $Comp
-L 2021-02-09_22-26-07:FERD2045SB-TR U5
+L bms_hardware-rescue:FERD2045SB-TR-2021-02-09_22-26-07 U5
 U 1 1 603F99FF
 P 6250 4500
+AR Path="/603F99FF" Ref="U5"  Part="1"
+AR Path="/60233007/603F99FF" Ref="U5"  Part="1"
 F 0 "U5" V 7156 4072 60  0000 R CNN
 F 1 "FERD2045SB-TR" V 7050 4072 60  0000 R CNN
@@
 $EndComp
 $Comp
-L Transistor_FET:IRF9310PbF Q13
+L bms_hardware-rescue:IRF9310PbF-Transistor_FET Q13
 U 1 1 603FB927
 P 6050 2700

Commit message: who knows
Parts:
- Q13: symbol bms_hardware-rescue:IRF9310PbF-Transistor_FET -> bms_hardware-rescue:IRF9310PbF-Transistor_FET-bms_hardware-rescue
- U5: symbol bms_hardware-rescue:FERD2045SB-TR-2021-02-09_22-26-07 -> bms_hardware-rescue:FERD2045SB-TR-2021-02-09_22-26-07-bms_hardware-rescue
Changed lines of the file:
@@
 	5800 4500 6150 4500
 $Comp
-L bms_hardware-rescue:FERD2045SB-TR-2021-02-09_22-26-07 U5
+L bms_hardware-rescue:FERD2045SB-TR-2021-02-09_22-26-07-bms_hardware-rescue U5
 U 1 1 603F99FF
 P 6250 4500
@@
 $EndComp
 $Comp
-L bms_hardware-rescue:IRF9310PbF-Transistor_FET Q13
+L bms_hardware-rescue:IRF9310PbF-Transistor_FET-bms_hardware-rescue Q13
 U 1 1 603FB927
 P 6050 2700
