File: balancing_module.sch (KiCad schematic (older format))
At the start: 54 parts, among them Q1 2N7002, Q2 2N7002, Q3 2N7002, Q4 2N7002, Q5 2N7002, Q6 2N7002

Commit message: Dletes hw_balanceo folder
Parts:
- removed R20, R33: R, Resistor_SMD:R_0805_2012Metric_Pad1.20x1.40mm_HandSolder, symbol Device:R
- added R23, R35: 47@1/2W, Resistor_SMD:R_1206_3216Metric_Pad1.30x1.75mm_HandSolder, symbol Device:R
- C13: renamed from C28; value C -> 0.1uF
- C14: renamed from C29; value C -> 0.1uF
- C15: renamed from C30; value C -> 0.1uF
- C19: renamed from C34; value C -> 0.1uF
- C20: renamed from C35; value C -> 0.1uF
- C21: renamed from C36; value C -> 0.1uF
- D1, D10, D11, D12, D2, D3, D4, D5, D6, D7, D8, D9: value D_Zener -> BZT52
- R15: renamed from R14; value R -> 1K
- R16: renamed from R15; value R -> 1K
- R17: renamed from R16; value R -> 1K
- R18: renamed from R17; value R -> 1M
- R19: renamed from R18; value R -> 1M
- R20: renamed from R19; value R -> 1M
- R21, R22, R34: value R -> 47@1/2W; footprint Resistor_SMD:R_0805_2012Metric_Pad1.20x1.40mm_HandSolder -> Resistor_SMD:R_1206_3216Metric_Pad1.30x1.75mm_HandSolder
- R27: renamed from R26; value R -> 1K
- R28: renamed from R27; value R -> 1K
- R29: renamed from R28; value R -> 1K
- R30: renamed from R29; value R -> 1M
- R31: renamed from R30; value R -> 1M
- R32: renamed from R31; value R -> 1M
- R33: renamed from R32; value R -> 47@1/2W; footprint Resistor_SMD:R_0805_2012Metric_Pad1.20x1.40mm_HandSolder -> Resistor_SMD:R_1206_3216Metric_Pad1.30x1.75mm_HandSolder
- renumbered C25 to C10, C26 to C11, C27 to C12, C31 to C16, C32 to C17, C33 to C18, R11 to R12, R12 to R13, R13 to R14, R23 to R24, R24 to R25, R25 to R26
Connections:
- net CELL_1+: now also R35.1; no longer R34.1
- net CELL_2+: now also R34.1
- net CELL_4+: now also R23.1; no longer R22.1
- net CELL_5+: now also R22.1; no longer R21.1
- net CELL_6+: now also R21.1
- net at Q1.3 (D): now also R21.2
- net at Q2.3 (D): now also R22.2; no longer R21.2
- net at Q3.3 (D): now also R23.2; no longer R22.2
- net at Q5.3 (D): now also R34.2
- net at Q6.3 (D): now also R35.2; no longer R34.2
Other:
- note added: "Avoid hot-plug transient voltages"
- note added: "anti-aliasing filter"
- moved on the sheet: D4
