File: can_hw.sch (KiCad schematic (older format))
At the start: 20 parts, among them J1 Conn_01x05, J2 Conn_01x05, U1 ADuM1201AR, U2 MCP2551-I-SN

Commit message: Final version pcb
Parts:
- removed C1, C3: 100nF, Capacitor_SMD:C_0805_2012Metric_Pad1.15x1.40mm_HandSolder, symbol adum:C
- removed C2: 330nF, Capacitor_SMD:C_0805_2012Metric_Pad1.15x1.40mm_HandSolder, symbol adum:C
- removed C4: 10uF, Capacitor_Tantalum_SMD:CP_EIA-6032-28_Kemet-C_Pad2.25x2.35mm_HandSolder, symbol adum:CP1
- removed D1, D2, D5: LED, LED_SMD:LED_0805_2012Metric, symbol adum:LED
- removed D3, D4: D, Diode_SMD:D_SOD-123, symbol adum:D
- removed J1, J2: Conn_01x05, Connector_JST:JST_EH_B5B-EH-A_1x05_P2.50mm_Vertical, symbol Connector_Generic:Conn_01x05
- removed JP1: Jumper_NO_Small, Jumper:SolderJumper-2_P1.3mm_Open_Pad1.0x1.5mm, symbol Default:Jumper_NO_Small
- removed PS1: PEP1-S5-D5-M, CONV_PEP1-S5-D5-M, symbol Can_Hw-rescue:PEP1-S5-D5-M-PEP1-S5-D5-M
- removed R1, R2: 1K5, Resistor_SMD:R_0805_2012Metric_Pad1.20x1.40mm_HandSolder, symbol adum:R
- removed R3: 0k, Resistor_SMD:R_0805_2012Metric_Pad1.20x1.40mm_HandSolder, symbol adum:R
- removed R4: 3K3, Resistor_SMD:R_0805_2012Metric_Pad1.20x1.40mm_HandSolder, symbol adum:R
- removed R5: 120, Resistor_SMD:R_0805_2012Metric_Pad1.20x1.40mm_HandSolder, symbol adum:R
- removed U2: MCP2551-I-SN, Package_SO:SOIC-8_3.9x4.9mm_P1.27mm, symbol Interface_CAN_LIN:MCP2551-I-SN
- added C59: 330nF, Capacitor_SMD:C_0805_2012Metric_Pad1.18x1.45mm_HandSolder, symbol Device:C
- added C60: 100nF, Capacitor_SMD:C_0805_2012Metric_Pad1.18x1.45mm_HandSolder, symbol Device:C
- added C61: 4.7uF, Capacitor_SMD:C_0805_2012Metric_Pad1.18x1.45mm_HandSolder, symbol Device:C
- added C62, C63: 100pF, Capacitor_SMD:C_0805_2012Metric_Pad1.18x1.45mm_HandSolder, symbol Device:C
- added J6: DB9_Male, Connector_Dsub:DSUB-9_Male_Horizontal_P2.77x2.84mm_EdgePinOffset4.94mm_Housed_MountingHolesOffset7.48mm, symbol Connector:DB9_Male
- added R5: 100, Resistor_SMD:R_0805_2012Metric_Pad1.20x1.40mm_HandSolder, symbol Device:R
- added R6, R7: 60, Resistor_SMD:R_0805_2012Metric_Pad1.20x1.40mm_HandSolder, symbol Device:R
- added U7: PDM1-S12-S3-S, CONV_PDM1-S12-S3-S, symbol Converter_DCDC:PDM1-S12-S3-S
- added U8: SN65HVD233, Package_SO:SOIC-8_3.9x4.9mm_P1.27mm, symbol Interface_CAN_LIN:SN65HVD233
Connections:
- net labels added: 3V3, CANH, CANL, CAN_RX, CAN_TX, ISO_3V3, ISO_CAN_RX, ISO_CAN_TX
- net labels removed: 3_3VCC_MCU, 5V_CAN, 5_VCC_MCU, CAN1_N, CAN1_P
- wire segments 84 -> 36
- no-connect marks 0 -> 6
Other:
- note removed: "SR Control \nResistor"
- note removed: "This Jumper is to connect the termination resistor \nIn case of the node is the last of the BUS"
- moved on the sheet: U1
