File: can_hw.sch (KiCad schematic (older format))
At the start: 12 parts, among them J6 DB9_Male, U1 ADuM1201AR, U7 PDM1-S12-S3-S, U8 SN65HVD233

Commit message: Edited sch page settings & printed schematic pdf
Parts:
- U7: symbol Converter_DCDC:PDM1-S12-S3-S -> bms_hardware-rescue:PDM1-S12-S3-S-Converter_DCDC
Changed lines of the file:
@@
 encoding utf-8
 Sheet 9 9
-Title ""
+Title "Battery Managment System (MBS)"
 Date ""
 Rev "A"
-Comp ""
+Comp "Ceccarelli Federico, Moya Martin,  Santos Lucio"
 Comment1 ""
-Comment2 ""
-Comment3 ""
-Comment4 ""
+Comment2 "Universidad Nacional de Rosario (UNR)"
+Comment3 "Facultad de Ciencias Exactas, Ingeniería y Agrimensura"
+Comment4 "Proyecto Final - Ingeniería Electrónica"
 $EndDescr
 Text HLabel 3300 3350 0    50   Input ~ 0
@@
 	2550 3150 2550 3200
 $Comp
-L Converter_DCDC:PDM1-S12-S3-S U7
+L bms_hardware-rescue:PDM1-S12-S3-S-Converter_DCDC U7
 U 1 1 60484510
 P 3900 2350
