File: vbat_3v3.sch (KiCad schematic (older format))
At the start: 15 parts

Commit message: Changes only global labels to main page
Connections:
- net GND renamed GND_BATT
Changed lines of the file:
@@
 $Descr A4 11693 8268
 encoding utf-8
-Sheet 7 7
+Sheet 6 7
 Title ""
 Date ""
@@
 	3150 2650 3150 2700
 Text HLabel 3150 3450 3    50   Input ~ 0
-GND
+GND_BATT
 Wire Wire Line
 	3150 3450 3150 3400
@@
 	750  3050 750  3100
 Text HLabel 750  3500 3    50   Input ~ 0
-GND
+GND_BATT
 Wire Wire Line
 	750  3450 750  3500
@@
 	5400 1650 5600 1650
 Text HLabel 5600 1750 3    50   Input ~ 0
-GND
+GND_BATT
 Wire Wire Line
 	5600 1650 5600 1750
@@
 V_IN
 Text HLabel 3250 1650 3    50   Input ~ 0
-GND
+GND_BATT
 Wire Wire Line
 	3850 800  3850 850
@@
 V_OUT
 Text HLabel 7450 1450 3    50   Input ~ 0
-GND
+GND_BATT
 Wire Wire Line
 	7450 1350 7450 1450

Commit message: Dletes hw_balanceo folder
Parts:
- gave numbers to parts that had none: 11
- renumbered R1 to R58, R2 to R59, R5 to R60, R6 to R61
Changed lines of the file:
@@
 $EndDescr
 $Comp
-L Regulator_Switching:TPS54331D U?
+L Regulator_Switching:TPS54331D U4
 U 1 1 60036491
 P 4700 1250
-F 0 "U?" H 4700 1920 50  0000 C CNN
+F 0 "U4" H 4700 1920 50  0000 C CNN
 F 1 "TPS54331D" H 4700 1829 50  0000 C CNN
 F 2 "Package_SO:SOIC-8_3.9x4.9mm_P1.27mm" H 4700 1250 50  0001 L BNN
@@
 $EndComp
 $Comp
-L Diode:B340 D?
+L Diode:B340 D19
 U 1 1 60048579
 P 1650 1350
-F 0 "D?" V 1696 1270 50  0000 R CNN
+F 0 "D19" V 1696 1270 50  0000 R CNN
 F 1 "B340" V 1605 1270 50  0000 R CNN
 F 2 "Diode_SMD:D_SMC" H 1650 1175 50  0001 C CNN
@@
 $EndComp
 $Comp
-L Device:C C?
+L Device:C C37
 U 1 1 6004918C
 P 2750 1400
-F 0 "C?" H 2865 1446 50  0000 L CNN
+F 0 "C37" H 2865 1446 50  0000 L CNN
 F 1 "330nF" H 2865 1355 50  0000 L CNN
 F 2 "Capacitor_SMD:C_0805_2012Metric_Pad1.18x1.45mm_HandSolder" H 2788 1250 50  0001 C CNN
@@
 $EndComp
 $Comp
-L Device:C C?
+L Device:C C38
 U 1 1 60049307
 P 3250 1400
-F 0 "C?" H 3365 1446 50  0000 L CNN
+F 0 "C38" H 3365 1446 50  0000 L CNN
 F 1 "10uF" H 3365 1355 50  0000 L CNN
 F 2 "Capacitor_SMD:C_0805_2012Metric_Pad1.18x1.45mm_HandSolder" H 3288 1250 50  0001 C CNN
@@
 $EndComp
 $Comp
-L Device:C C?
+L Device:C C42
 U 1 1 600495AA
 P 7450 1200
-F 0 "C?" H 7565 1246 50  0000 L CNN
+F 0 "C42" H 7565 1246 50  0000 L CNN
 F 1 "10uF" H 7565 1155 50  0000 L CNN
 F 2 "Capacitor_SMD:C_0805_2012Metric_Pad1.18x1.45mm_HandSolder" H 7488 1050 50  0001 C CNN
@@
 $EndComp
 $Comp
-L Device:C C?
+L Device:C C40
 U 1 1 60049A2E
 P 5400 1000
-F 0 "C?" H 5515 1046 50  0000 L CNN
+F 0 "C40" H 5515 1046 50  0000 L CNN
 F 1 "2.2nF" H 5515 955 50  0000 L CNN
 F 2 "Capacitor_SMD:C_0805_2012Metric_Pad1.18x1.45mm_HandSolder" H 5438 850 50  0001 C CNN
@@
 $EndComp
 $Comp
-L Device:C C?
+L Device:C C41
 U 1 1 60049CF6
 P 5800 1300
-F 0 "C?" H 5915 1346 50  0000 L CNN
+F 0 "C41" H 5915 1346 50  0000 L CNN
 F 1 "1nF" H 5915 1255 50  0000 L CNN
 F 2 "Capacitor_SMD:C_0805_2012Metric_Pad1.18x1.45mm_HandSolder" H 5838 1150 50  0001 C CNN
@@
 $EndComp
 $Comp
-L Device:R R5
+L Device:R R60
 U 1 1 6004A339
 P 3150 2850
-F 0 "R5" H 3220 2896 50  0000 L CNN
+F 0 "R60" H 3220 2896 50  0000 L CNN
 F 1 "9K1" H 3220 2805 50  0000 L CNN
 F 2 "Resistor_SMD:R_0805_2012Metric_Pad1.20x1.40mm_HandSolder" V 3080 2850 50  0001 C CNN
@@
 $EndComp
 $Comp
-L Device:R R6
+L Device:R R61
 U 1 1 6004A5D5
 P 3150 3250
-F 0 "R6" H 3220 3296 50  0000 L CNN
+F 0 "R61" H 3220 3296 50  0000 L CNN
 F 1 "1K8" H 3220 3205 50  0000 L CNN
 F 2 "Resistor_SMD:R_0805_2012Metric_Pad1.20x1.40mm_HandSolder" V 3080 3250 50  0001 C CNN
@@
 $EndComp
 $Comp
-L Device:R R2
+L Device:R R59
 U 1 1 6004A934
 P 750 3300
-F 0 "R2" H 820 3346 50  0000 L CNN
+F 0 "R59" H 820 3346 50  0000 L CNN
 F 1 "27K" H 820 3255 50  0000 L CNN
 F 2 "Resistor_SMD:R_0805_2012Metric_Pad1.20x1.40mm_HandSolder" V 680 3300 50  0001 C CNN
@@
 $EndComp
 $Comp
-L Device:R R1
+L Device:R R58
 U 1 1 6004ABA6
 P 750 2900
-F 0 "R1" H 820 2946 50  0000 L CNN
+F 0 "R58" H 820 2946 50  0000 L CNN
 F 1 "330K" H 820 2855 50  0000 L CNN
 F 2 "Resistor_SMD:R_0805_2012Metric_Pad1.20x1.40mm_HandSolder" V 680 2900 50  0001 C CNN
@@
 $EndComp
 $Comp
-L Device:R R?
+L Device:R R62
 U 1 1 6004AED7
 P 5400 1500
-F 0 "R?" H 5470 1546 50  0000 L CNN
+F 0 "R62" H 5470 1546 50  0000 L CNN
 F 1 "5K1" H 5470 1455 50  0000 L CNN
 F 2 "" V 5330 1500 50  0001 C CNN
@@
 $EndComp
 $Comp
-L Device:L L?
+L Device:L L2
 U 1 1 60057BAE
 P 7200 950
-F 0 "L?" V 7019 950 50  0000 C CNN
+F 0 "L2" V 7019 950 50  0000 C CNN
 F 1 "6.8uH" V 7110 950 50  0000 C CNN
 F 2 "BOURNS_SRP6030VA:SRP6030VA-6R8M" H 7200 950 50  0001 C CNN
@@
 PH
 $Comp
-L Device:C C?
+L Device:C C39
 U 1 1 60049780
 P 3300 950
-F 0 "C?" H 3415 996 50  0000 L CNN
+F 0 "C39" H 3415 996 50  0000 L CNN
 F 1 "0.1uF" H 3415 905 50  0000 L CNN
 F 2 "Capacitor_SMD:C_0805_2012Metric_Pad1.18x1.45mm_HandSolder" H 3338 800 50  0001 C CNN
@@
 $EndComp
 $Comp
-L Device:C C?
+L Device:C C36
 U 1 1 60056C6C
 P 2050 1350
-F 0 "C?" H 2165 1396 50  0000 L CNN
+F 0 "C36" H 2165 1396 50  0000 L CNN
 F 1 "3.3nF" H 2165 1305 50  0000 L CNN
 F 2 "Capacitor_SMD:C_0805_2012Metric_Pad1.18x1.45mm_HandSolder" H 2088 1200 50  0001 C CNN

Commit message: Fixes missing footprints, adds initial pcb
Parts:
- L2: footprint BOURNS_SRP6030VA:SRP6030VA-6R8M -> Inductor_SMD:L_BOURNS_SRP6030
- R62: footprint (none) -> Resistor_SMD:R_0805_2012Metric_Pad1.20x1.40mm_HandSolder
Changed lines of the file:
@@
 F 0 "R62" H 5470 1546 50  0000 L CNN
 F 1 "5K1" H 5470 1455 50  0000 L CNN
-F 2 "" V 5330 1500 50  0001 C CNN
+F 2 "Resistor_SMD:R_0805_2012Metric_Pad1.20x1.40mm_HandSolder" V 5330 1500 50  0001 C CNN
 F 3 "~" H 5400 1500 50  0001 C CNN
 	1    5400 1500
@@
 F 0 "L2" V 7019 950 50  0000 C CNN
 F 1 "6.8uH" V 7110 950 50  0000 C CNN
-F 2 "BOURNS_SRP6030VA:SRP6030VA-6R8M" H 7200 950 50  0001 C CNN
+F 2 "Inductor_SMD:L_BOURNS_SRP6030" H 7200 950 50  0001 C CNN
 F 3 "https://ar.mouser.com/ProductDetail/SRP6030VA-6R8M" H 7200 950 50  0001 C CNN
 	1    7200 950

Commit message: Added mouser reference.com to charger imput molex pin
Parts:
- U4: symbol Regulator_Switching:TPS54331D -> bms_hardware-rescue:TPS54331D-Regulator_Switching
Changed lines of the file:
@@
 $EndDescr
 $Comp
-L Regulator_Switching:TPS54331D U4
+L bms_hardware-rescue:TPS54331D-Regulator_Switching U4
 U 1 1 60036491
 P 4700 1250

Commit message: Final version pcb
Parts:
- removed U4: TPS54331D, Package_SO:SOIC-8_3.9x4.9mm_P1.27mm, symbol bms_hardware-rescue:TPS54331D-Regulator_Switching
- added U4: TPS54331D, Package_SO:SOIC-8_3.9x4.9mm_P1.27mm, symbol Regulator_Switching:TPS54331D
Connections:
- net EN: now also U4.3 (EN)
- net GND_BATT: now also U4.7 (GND)
- net PH: now also U4.8 (PH)
- net VSENSE: now also U4.5 (VSENSE)
- net V_IN: now also U4.2 (VIN)
- net at C39.1: now also U4.1 (BOOT)
- net at C36.1: now also U4.4 (SS)
- net at C40.1, C41.1: now also U4.6 (COMP)
Changed lines of the file:
@@
 $Descr A4 11693 8268
 encoding utf-8
-Sheet 6 8
+Sheet 6 9
 Title ""
 Date ""
@@
 $EndDescr
 $Comp
-L bms_hardware-rescue:TPS54331D-Regulator_Switching U4
-U 1 1 60036491
-P 4700 1250
-F 0 "U4" H 4700 1920 50  0000 C CNN
-F 1 "TPS54331D" H 4700 1829 50  0000 C CNN
-F 2 "Package_SO:SOIC-8_3.9x4.9mm_P1.27mm" H 4700 1250 50  0001 L BNN
-F 3 "https://ar.mouser.com/ProductDetail/Texas-Instruments/TPS54331DR/?qs=QyYHynRG50rsSYcB%2Ftz4Yw%3D%3D" H 4700 1250 50  0001 L BNN
-	1    4700 1250
-	1    0    0    -1
-$EndComp
-$Comp
 L Diode:B340 D19
 U 1 1 60048579
@@
 Wire Wire Line
 	5400 850  5800 850
-Connection ~ 5400 850
-Connection ~ 5400 1650
 Wire Wire Line
 	5400 1150 5400 1350
@@
 Wire Notes Line
 	11100 650  11100 1700
+$Comp
+L Regulator_Switching:TPS54331D U4
+U 1 1 603F4701
+P 4700 1250
+F 0 "U4" H 4700 1920 50  0000 C CNN
+F 1 "TPS54331D" H 4700 1829 50  0000 C CNN
+F 2 "Package_SO:SOIC-8_3.9x4.9mm_P1.27mm" H 4700 1250 50  0001 L BNN
+F 3 "https://ar.mouser.com/ProductDetail/Texas-Instruments/TPS54331DR/?qs=QyYHynRG50rsSYcB%2Ftz4Yw%3D%3D" H 4700 1250 50  0001 L BNN
+	1    4700 1250
+	1    0    0    -1
+$EndComp
+Connection ~ 5400 850
+Connection ~ 5400 1650
 $EndSCHEMATC
