File: vbat_3v3.sch (KiCad schematic (older format))
At the start: 15 parts, among them U4 TPS54331D

Commit message: Edited sch page settings & printed schematic pdf
Parts:
- U4: symbol Regulator_Switching:TPS54331D -> bms_hardware-rescue:TPS54331D-Regulator_Switching
Changed lines of the file:
@@
 encoding utf-8
 Sheet 6 9
-Title ""
+Title "Battery Managment System (MBS)"
 Date ""
 Rev "A"
-Comp ""
+Comp "Ceccarelli Federico, Moya Martin,  Santos Lucio"
 Comment1 ""
-Comment2 ""
-Comment3 ""
-Comment4 ""
+Comment2 "Universidad Nacional de Rosario (UNR)"
+Comment3 "Facultad de Ciencias Exactas, Ingeniería y Agrimensura"
+Comment4 "Proyecto Final - Ingeniería Electrónica"
 $EndDescr
 $Comp
@@
 	11100 650  11100 1700
 $Comp
-L Regulator_Switching:TPS54331D U4
+L bms_hardware-rescue:TPS54331D-Regulator_Switching U4
 U 1 1 603F4701
 P 4700 1250

Commit message: who knows
Parts:
- U4: symbol bms_hardware-rescue:TPS54331D-Regulator_Switching -> bms_hardware-rescue:TPS54331D-Regulator_Switching-bms_hardware-rescue
Changed lines of the file:
@@
 	11100 650  11100 1700
 $Comp
-L bms_hardware-rescue:TPS54331D-Regulator_Switching U4
+L bms_hardware-rescue:TPS54331D-Regulator_Switching-bms_hardware-rescue U4
 U 1 1 603F4701
 P 4700 1250
