File: bat_charger.sch (KiCad schematic (older format))
At the start: 59 parts, among them J3 Vcc In, J4 CH_TS, Q10 FDD86580-F085, Q7 Q_PMOS_GDS, Q8 Q_PMOS_GDS, Q9 FDD86580-F085, SW1 Reset, SW2 Select CE, U4 BQ24618RGET

Commit message: Adds Can Pins
Parts:
- Q7, Q8: value Q_PMOS_GDS -> DMP4051LK3
Changed lines of the file:
@@
 P 4050 1400
 F 0 "Q8" V 4392 1400 50  0000 C CNN
-F 1 "Q_PMOS_GDS" V 4301 1400 50  0000 C CNN
+F 1 "DMP4051LK3" V 4301 1400 50  0000 C CNN
 F 2 "TO_SOT_Packages_SMD:TO-252-2_Rectifier" H 4250 1500 50  0001 C CNN
 F 3 "https://ar.mouser.com/ProductDetail/DMP4051LK3-13" H 4050 1400 50  0001 C CNN
@@
 P 3150 1400
 F 0 "Q7" V 3399 1400 50  0000 C CNN
-F 1 "Q_PMOS_GDS" V 3490 1400 50  0000 C CNN
+F 1 "DMP4051LK3" V 3490 1400 50  0000 C CNN
 F 2 "TO_SOT_Packages_SMD:TO-252-2_Rectifier" H 3350 1500 50  0001 C CNN
 F 3 "https://ar.mouser.com/ProductDetail/DMP4051LK3-13" H 3150 1400 50  0001 C CNN

Commit message: Dletes hw_balanceo folder
Parts:
- J3: renamed from J4; footprint Connector_JST:JST_XH_S7B-XH-A_1x07_P2.50mm_Horizontal -> Connector_JST:JST_XH_S2B-XH-A_1x02_P2.50mm_Horizontal
- R40: renamed from R43; footprint Resistors_SMD:R_0805_HandSoldering -> Resistor_SMD:R_0805_2012Metric_Pad1.20x1.40mm_HandSolder
- R41: renamed from R44; footprint Resistors_SMD:R_0805_HandSoldering -> Resistor_SMD:R_0805_2012Metric_Pad1.20x1.40mm_HandSolder
- R42: renamed from R45; footprint Resistors_SMD:R_0805_HandSoldering -> Resistor_SMD:R_0805_2012Metric_Pad1.20x1.40mm_HandSolder
- R43: renamed from R46; footprint Resistors_SMD:R_0805_HandSoldering -> Resistor_SMD:R_0805_2012Metric_Pad1.20x1.40mm_HandSolder
- R44: renamed from R47; footprint Resistors_SMD:R_0805_HandSoldering -> Resistor_SMD:R_0805_2012Metric_Pad1.20x1.40mm_HandSolder
- R45: renamed from R48; footprint Resistors_SMD:R_0805_HandSoldering -> Resistor_SMD:R_0805_2012Metric_Pad1.20x1.40mm_HandSolder
- R46: renamed from R49; footprint Resistors_SMD:R_0805_HandSoldering -> Resistor_SMD:R_0805_2012Metric_Pad1.20x1.40mm_HandSolder
- R47: renamed from R50; footprint Resistors_SMD:R_0805_HandSoldering -> Resistor_SMD:R_0805_2012Metric_Pad1.20x1.40mm_HandSolder
- R48: renamed from R51; footprint Resistors_SMD:R_0805_HandSoldering -> Resistor_SMD:R_0805_2012Metric_Pad1.20x1.40mm_HandSolder
- R49: renamed from R52; footprint Resistors_SMD:R_0805_HandSoldering -> Resistor_SMD:R_0805_2012Metric_Pad1.20x1.40mm_HandSolder
- R50: renamed from R53; footprint Resistors_SMD:R_0805_HandSoldering -> Resistor_SMD:R_0805_2012Metric_Pad1.20x1.40mm_HandSolder
- R51: renamed from R54; footprint Resistors_SMD:R_0805_HandSoldering -> Resistor_SMD:R_0805_2012Metric_Pad1.20x1.40mm_HandSolder
- R53: renamed from R56; footprint Resistors_SMD:R_0805_HandSoldering -> Resistor_SMD:R_0805_2012Metric_Pad1.20x1.40mm_HandSolder
- R54: renamed from R57; footprint Resistors_SMD:R_0805_HandSoldering -> Resistor_SMD:R_0805_2012Metric_Pad1.20x1.40mm_HandSolder
- R55: renamed from R58; footprint Resistors_SMD:R_0805_HandSoldering -> Resistor_SMD:R_0805_2012Metric_Pad1.20x1.40mm_HandSolder
- R56: renamed from R59; footprint Resistors_SMD:R_0805_HandSoldering -> Resistor_SMD:R_0805_2012Metric_Pad1.20x1.40mm_HandSolder
- R57: renamed from R60; footprint Resistors_SMD:R_0805_HandSoldering -> Resistor_SMD:R_0805_2012Metric_Pad1.20x1.40mm_HandSolder
- renumbered C38 to C22, C39 to C23, C40 to C24, C41 to C25, C42 to C26, C43 to C27, C44 to C28, C45 to C29, C46 to C30, C47 to C31, C48 to C32, C49 to C33, C50 to C34, C51 to C35, J3 to J2, L2 to L1, R39 to R36, R40 to R37, R41 to R38, R42 to R39, R55 to R52, U4 to U3

Commit message: Adds bat_switch to main sheet
Parts:
- C25, C26, C27, C31, C32, C33: footprint Capacitors_SMD:C_0805_HandSoldering -> Capacitor_SMD:C_0805_2012Metric_Pad1.18x1.45mm_HandSolder
Changed lines of the file:
@@
 $Descr A4 11693 8268
 encoding utf-8
-Sheet 5 7
+Sheet 5 8
 Title ""
 Date ""
@@
 F 0 "C25" H 3300 3600 50  0000 R CNN
 F 1 "0.1uF" H 3400 3800 50  0000 R CNN
-F 2 "Capacitors_SMD:C_0805_HandSoldering" H 3188 3550 50  0001 C CNN
+F 2 "Capacitor_SMD:C_0805_2012Metric_Pad1.18x1.45mm_HandSolder" H 3188 3550 50  0001 C CNN
 F 3 "https://ar.mouser.com/ProductDetail/581-08055C104K/" H 3150 3700 50  0001 C CNN
 	1    3150 3700
@@
 F 0 "C33" H 7300 4400 50  0000 R CNN
 F 1 "0.1uF" H 7300 4600 50  0000 R CNN
-F 2 "Capacitors_SMD:C_0805_HandSoldering" H 7388 4350 50  0001 C CNN
+F 2 "Capacitor_SMD:C_0805_2012Metric_Pad1.18x1.45mm_HandSolder" H 7388 4350 50  0001 C CNN
 F 3 "https://ar.mouser.com/ProductDetail/581-08055C104K/" H 7350 4500 50  0001 C CNN
 	1    7350 4500
@@
 F 0 "C26" H 3100 4250 50  0000 R CNN
 F 1 "0.1uF" H 3100 4050 50  0000 R CNN
-F 2 "Capacitors_SMD:C_0805_HandSoldering" H 3188 4000 50  0001 C CNN
+F 2 "Capacitor_SMD:C_0805_2012Metric_Pad1.18x1.45mm_HandSolder" H 3188 4000 50  0001 C CNN
 F 3 "https://ar.mouser.com/ProductDetail/581-08055C104K/" H 3150 4150 50  0001 C CNN
 	1    3150 4150
@@
 F 0 "C31" V 7602 3550 50  0000 C CNN
 F 1 "0.1uF" V 7511 3550 50  0000 C CNN
-F 2 "Capacitors_SMD:C_0805_HandSoldering" H 7388 3400 50  0001 C CNN
+F 2 "Capacitor_SMD:C_0805_2012Metric_Pad1.18x1.45mm_HandSolder" H 7388 3400 50  0001 C CNN
 F 3 "https://ar.mouser.com/ProductDetail/581-08055C104K/" H 7350 3550 50  0001 C CNN
 	1    7350 3550
@@
 F 0 "C32" H 7465 4146 50  0000 L CNN
 F 1 "0.1uF" H 7465 4055 50  0000 L CNN
-F 2 "Capacitors_SMD:C_0805_HandSoldering" H 7388 3950 50  0001 C CNN
+F 2 "Capacitor_SMD:C_0805_2012Metric_Pad1.18x1.45mm_HandSolder" H 7388 3950 50  0001 C CNN
 F 3 "https://ar.mouser.com/ProductDetail/581-08055C104K/" H 7350 4100 50  0001 C CNN
 	1    7350 4100
@@
 F 0 "C27" H 3815 1454 50  0000 L CNN
 F 1 "0.1uF" H 3815 1545 50  0000 L CNN
-F 2 "Capacitors_SMD:C_0805_HandSoldering" H 3738 1350 50  0001 C CNN
+F 2 "Capacitor_SMD:C_0805_2012Metric_Pad1.18x1.45mm_HandSolder" H 3738 1350 50  0001 C CNN
 F 3 "https://ar.mouser.com/ProductDetail/581-08055C104K/" H 3700 1500 50  0001 C CNN
 	1    3700 1500

Commit message: Fixes missing footprints, adds initial pcb
Parts:
- C22, C23, C24, C28, C30: footprint Capacitors_SMD:C_0805_HandSoldering -> Capacitor_SMD:C_0805_2012Metric_Pad1.18x1.45mm_HandSolder
- C29, C34, C35: footprint Capacitors_SMD:CP_Elec_6.3x7.7 -> Capacitor_SMD:C_Elec_6.3x7.7
- D13: footprint Diodes_THT:D_A-405_P7.62mm_Horizontal -> Diode_THT:D_A-405_P7.62mm_Horizontal
- D14, D15, D16, D17: footprint LEDs:LED_0603_HandSoldering -> LED_SMD:LED_0603_1608Metric_Pad1.05x0.95mm_HandSolder
- D18: footprint Diodes_SMD:D_SOD-523 -> Diode_SMD:D_SOD-523
- J3: renamed from J2; footprint Connectors_Molex:Molex_KK-41791-02_02x3.96mm_Straight -> Connector_Molex:Molex_KK-396_A-41791-0002_1x02_P3.96mm_Vertical
- L1: footprint BOURNS_SRP6030VA:SRP6030VA-6R8M -> Inductor_SMD:L_BOURNS_SRP6030
- NT1: footprint Oddities:NetTie-I_Connected_SMD -> NetTie:NetTie-3_SMD_Pad0.5mm
- Q10, Q7, Q8, Q9: footprint TO_SOT_Packages_SMD:TO-252-2_Rectifier -> Package_TO_SOT_SMD:TO-252-2
- R36, R37: footprint Resistors_SMD:R_0805_HandSoldering -> Resistor_SMD:R_0805_2012Metric_Pad1.20x1.40mm_HandSolder
- R38, R39, R52: footprint Resistors_SMD:R_1206_HandSoldering -> Resistor_SMD:R_1206_3216Metric_Pad1.30x1.75mm_HandSolder
- SW1: footprint Buttons_Switches_THT:SW_TH_Tactile_Omron_B3F-10xx -> Button_Switch_THT:SW_TH_Tactile_Omron_B3F-10xx
- SW2: footprint Buttons_Switches_THT:SW_DIP_x2_W7.62mm_Piano -> Button_Switch_THT:SW_DIP_SPSTx02_Slide_6.7x6.64mm_W7.62mm_P2.54mm_LowProfile
- TP1, TP2, TP3, TP4, TP5, TP6: footprint Keystone_5016:KEYSTONE_5016 -> TestPoint:KEYSTONE_5016
- U3: footprint lib:BQ24618RGET -> Package_DFN_QFN:VQFN-24-1EP_4x4mm_P0.5mm_EP2.45x2.45mm
- renumbered J3 to J4
Other:
- moved on the sheet: U3A, U3B

Commit message: Added mouser reference.com to charger imput molex pin
Connections:
- net labels added: CE_BQ24, PG_BQ24, STAT1_BQ24, STAT2_BQ24
- net labels removed: uCE
Other:
- moved on the sheet: D14, D15, D16, D17, R44, R45, R46, R47, TP5
Changed lines of the file:
@@
 L Device:LED D14
 U 1 1 5FC6CF41
-P 5150 7050
-F 0 "D14" V 5189 6932 50  0000 R CNN
-F 1 "VCC" V 5098 6932 50  0000 R CNN
-F 2 "LED_SMD:LED_0603_1608Metric_Pad1.05x0.95mm_HandSolder" H 5150 7050 50  0001 C CNN
-F 3 "https://ar.mouser.com/ProductDetail/LTST-C190KGKT" H 5150 7050 50  0001 C CNN
-	1    5150 7050
+P 4850 7050
+F 0 "D14" V 4889 6932 50  0000 R CNN
+F 1 "VCC" V 4798 6932 50  0000 R CNN
+F 2 "LED_SMD:LED_0603_1608Metric_Pad1.05x0.95mm_HandSolder" H 4850 7050 50  0001 C CNN
+F 3 "https://ar.mouser.com/ProductDetail/LTST-C190KGKT" H 4850 7050 50  0001 C CNN
+	1    4850 7050
 	0    -1   -1   0
 $EndComp
@@
 L Device:R R44
 U 1 1 5FC6E27D
-P 5150 6600
-F 0 "R44" H 5220 6646 50  0000 L CNN
-F 1 "5K6" H 5220 6555 50  0000 L CNN
-F 2 "Resistor_SMD:R_0805_2012Metric_Pad1.20x1.40mm_HandSolder" V 5080 6600 50  0001 C CNN
-F 3 "https://ar.mouser.com/ProductDetail/ERJ-T06J562V" H 5150 6600 50  0001 C CNN
-	1    5150 6600
-	1    0    0    -1
-$EndComp
-Wire Wire Line
-	5150 7500 5150 7200
-Wire Wire Line
-	5150 6900 5150 6750
-Wire Wire Line
-	5150 6450 5150 6250
+P 4850 6600
+F 0 "R44" H 4920 6646 50  0000 L CNN
+F 1 "5K6" H 4920 6555 50  0000 L CNN
+F 2 "Resistor_SMD:R_0805_2012Metric_Pad1.20x1.40mm_HandSolder" V 4780 6600 50  0001 C CNN
+F 3 "https://ar.mouser.com/ProductDetail/ERJ-T06J562V" H 4850 6600 50  0001 C CNN
+	1    4850 6600
+	1    0    0    -1
+$EndComp
+Wire Wire Line
+	4850 7500 4850 7200
+Wire Wire Line
+	4850 6900 4850 6750
+Wire Wire Line
+	4850 6450 4850 6250
 Text Label 4050 4450 2    50   ~ 0
 STAT1
@@
 STAT2
 Wire Wire Line
-	6250 6900 6250 6750
-Wire Wire Line
-	6250 7200 6250 7300
+	6050 6900 6050 6750
+Wire Wire Line
+	6050 7200 6050 7300
 Wire Wire Line
 	4050 4450 3800 4450
@@
 ACDRV
 Wire Wire Line
-	6250 7300 6500 7300
-Wire Wire Line
-	5900 7400 6200 7400
-Wire Wire Line
-	5900 7200 5900 7400
-Text Label 6500 7300 2    50   ~ 0
+	6050 7300 6300 7300
+Wire Wire Line
+	5700 7400 6000 7400
+Wire Wire Line
+	5700 7200 5700 7400
+Text Label 6300 7300 2    50   ~ 0
 STAT1
-Text Label 6200 7400 2    50   ~ 0
+Text Label 6000 7400 2    50   ~ 0
 STAT2
 Wire Wire Line
-	5550 7200 5550 7500
-Wire Wire Line
-	5550 7500 5700 7500
-Text Label 5700 7500 2    50   ~ 0
+	5350 7200 5350 7500
+Wire Wire Line
+	5350 7500 5500 7500
+Text Label 5500 7500 2    50   ~ 0
 PG
 Wire Wire Line
-	5550 6900 5550 6750
-Text HLabel 6500 7300 2    50   Output ~ 0
-STAT1
-Text HLabel 6200 7400 2    50   Output ~ 0
-STAT2
-Text HLabel 5700 7500 2    50   Output ~ 0
-PG
+	5350 6900 5350 6750
+Text HLabel 6300 7300 2    50   Output ~ 0
+STAT1_BQ24
+Text HLabel 6000 7400 2    50   Output ~ 0
+STAT2_BQ24
+Text HLabel 5500 7500 2    50   Output ~ 0
+PG_BQ24
 $Comp
 L Device:LED D15
 U 1 1 5FE43B78
-P 5550 6600
-F 0 "D15" V 5550 6500 50  0000 R CNN
-F 1 "PG" V 5650 6500 50  0000 R CNN
-F 2 "LED_SMD:LED_0603_1608Metric_Pad1.05x0.95mm_HandSolder" H 5550 6600 50  0001 C CNN
-F 3 "https://ar.mouser.com/ProductDetail/LTST-C190KGKT" H 5550 6600 50  0001 C CNN
-	1    5550 6600
+P 5350 6600
+F 0 "D15" V 5350 6500 50  0000 R CNN
+F 1 "PG" V 5450 6500 50  0000 R CNN
+F 2 "LED_SMD:LED_0603_1608Metric_Pad1.05x0.95mm_HandSolder" H 5350 6600 50  0001 C CNN
+F 3 "https://ar.mouser.com/ProductDetail/LTST-C190KGKT" H 5350 6600 50  0001 C CNN
+	1    5350 6600
 	0    -1   -1   0
 $EndComp
 Wire Wire Line
-	5900 6900 5900 6750
-Wire Wire Line
-	5550 6450 5550 6300
-Wire Wire Line
-	5550 6300 5900 6300
-Wire Wire Line
-	5900 6300 6250 6300
-Wire Wire Line
-	6250 6300 6250 6450
-Connection ~ 5900 6300
-Wire Wire Line
-	5900 6450 5900 6300
+	5700 6900 5700 6750
+Wire Wire Line
+	5350 6450 5350 6300
+Wire Wire Line
+	5350 6300 5700 6300
+Wire Wire Line
+	5700 6300 6050 6300
+Wire Wire Line
+	6050 6300 6050 6450
+Connection ~ 5700 6300
+Wire Wire Line
+	5700 6450 5700 6300
 $Comp
 L Device:R R45
 U 1 1 5FDF3D4E
-P 5550 7050
-F 0 "R45" H 5480 7004 50  0000 R CNN
-F 1 "470R" H 5480 7095 50  0000 R CNN
-F 2 "Resistor_SMD:R_0805_2012Metric_Pad1.20x1.40mm_HandSolder" V 5480 7050 50  0001 C CNN
-F 3 "https://ar.mouser.com/ProductDetail/CR0805-FX-4220ELF" H 5550 7050 50  0001 C CNN
-	1    5550 7050
+P 5350 7050
+F 0 "R45" H 5280 7004 50  0000 R CNN
+F 1 "470R" H 5280 7095 50  0000 R CNN
+F 2 "Resistor_SMD:R_0805_2012Metric_Pad1.20x1.40mm_HandSolder" V 5280 7050 50  0001 C CNN
+F 3 "https://ar.mouser.com/ProductDetail/CR0805-FX-4220ELF" H 5350 7050 50  0001 C CNN
+	1    5350 7050
 	-1   0    0    1
 $EndComp
@@
 L Device:R R46
 U 1 1 5FD06754
-P 5900 7050
-F 0 "R46" H 5830 7004 50  0000 R CNN
-F 1 "470R" H 5830 7095 50  0000 R CNN
-F 2 "Resistor_SMD:R_0805_2012Metric_Pad1.20x1.40mm_HandSolder" V 5830 7050 50  0001 C CNN
-F 3 "https://ar.mouser.com/ProductDetail/CR0805-FX-4220ELF" H 5900 7050 50  0001 C CNN
-	1    5900 7050
+P 5700 7050
+F 0 "R46" H 5630 7004 50  0000 R CNN
+F 1 "470R" H 5630 7095 50  0000 R CNN
+F 2 "Resistor_SMD:R_0805_2012Metric_Pad1.20x1.40mm_HandSolder" V 5630 7050 50  0001 C CNN
+F 3 "https://ar.mouser.com/ProductDetail/CR0805-FX-4220ELF" H 5700 7050 50  0001 C CNN
+	1    5700 7050
 	-1   0    0    1
 $EndComp
@@
 L Device:R R47
 U 1 1 5FD04CAC
-P 6250 7050
-F 0 "R47" H 6180 7004 50  0000 R CNN
-F 1 "470R" H 6180 7095 50  0000 R CNN
-F 2 "Resistor_SMD:R_0805_2012Metric_Pad1.20x1.40mm_HandSolder" V 6180 7050 50  0001 C CNN
-F 3 "https://ar.mouser.com/ProductDetail/CR0805-FX-4220ELF" H 6250 7050 50  0001 C CNN
-	1    6250 7050
+P 6050 7050
+F 0 "R47" H 5980 7004 50  0000 R CNN
+F 1 "470R" H 5980 7095 50  0000 R CNN
+F 2 "Resistor_SMD:R_0805_2012Metric_Pad1.20x1.40mm_HandSolder" V 5980 7050 50  0001 C CNN
+F 3 "https://ar.mouser.com/ProductDetail/CR0805-FX-4220ELF" H 6050 7050 50  0001 C CNN
+	1    6050 7050
 	-1   0    0    1
 $EndComp
@@
 L Device:LED D17
 U 1 1 5FE36851
-P 6250 6600
-F 0 "D17" V 6250 6500 50  0000 R CNN
-F 1 "STAT1" V 6350 6550 50  0000 R CNN
-F 2 "LED_SMD:LED_0603_1608Metric_Pad1.05x0.95mm_HandSolder" H 6250 6600 50  0001 C CNN
-F 3 "https://mouser.com/ProductDetail/LTST-C190AKT" H 6250 6600 50  0001 C CNN
-	1    6250 6600
+P 6050 6600
+F 0 "D17" V 6050 6500 50  0000 R CNN
+F 1 "STAT1" V 6150 6550 50  0000 R CNN
+F 2 "LED_SMD:LED_0603_1608Metric_Pad1.05x0.95mm_HandSolder" H 6050 6600 50  0001 C CNN
+F 3 "https://mouser.com/ProductDetail/LTST-C190AKT" H 6050 6600 50  0001 C CNN
+	1    6050 6600
 	0    -1   -1   0
 $EndComp
@@
 L Device:LED D16
 U 1 1 5FE4380E
-P 5900 6600
-F 0 "D16" V 5900 6500 50  0000 R CNN
-F 1 "STAT2" V 6000 6550 50  0000 R CNN
-F 2 "LED_SMD:LED_0603_1608Metric_Pad1.05x0.95mm_HandSolder" H 5900 6600 50  0001 C CNN
-F 3 "https://ar.mouser.com/ProductDetail/LTST-C190AKT" H 5900 6600 50  0001 C CNN
-	1    5900 6600
+P 5700 6600
+F 0 "D16" V 5700 6500 50  0000 R CNN
+F 1 "STAT2" V 5800 6550 50  0000 R CNN
+F 2 "LED_SMD:LED_0603_1608Metric_Pad1.05x0.95mm_HandSolder" H 5700 6600 50  0001 C CNN
+F 3 "https://ar.mouser.com/ProductDetail/LTST-C190AKT" H 5700 6600 50  0001 C CNN
+	1    5700 6600
 	0    -1   -1   0
 $EndComp
@@
 	6900 7700 6900 5650
 Wire Notes Line
-	6900 5650 4750 5650
-Wire Notes Line
-	4750 5650 4750 7700
-Wire Notes Line
-	4750 7700 6900 7700
+	6900 5650 4450 5650
+Wire Notes Line
+	4450 5650 4450 7700
+Wire Notes Line
+	4450 7700 6900 7700
 Text Label 9950 5150 0    50   ~ 0
 VFB
@@
 F 1 "Vcc In" H 1830 1791 50  0000 L CNN
 F 2 "Connector_Molex:Molex_KK-396_A-41791-0002_1x02_P3.96mm_Vertical" H 1750 1800 50  0001 C CNN
-F 3 "~" H 1750 1800 50  0001 C CNN
+F 3 "https://www.mouser.com/ProductDetail/571-1744429-2/" H 1750 1800 50  0001 C CNN
 	1    1750 1800
 	-1   0    0    1
@@
 Wire Wire Line
 	4050 4250 3800 4250
-Text Notes 5500 5800 0    59   ~ 12
+Text Notes 5300 5800 0    59   ~ 12
 Status LEDs & Signals
-Text Notes 750  3550 0    59   ~ 12
+Text Notes 650  3550 0    59   ~ 12
 Reset & CE Source Selector
 Wire Notes Line
-	650  5600 650  3400
+	550  5600 550  3400
 Wire Notes Line
 	2050 3400 2050 5600
 Wire Notes Line
-	650  3400 2050 3400
+	550  3400 2050 3400
 Wire Wire Line
 	1750 5150 1750 5200
@@
 	1000 5100 1100 5100
 Text HLabel 1000 5200 0    50   Input ~ 0
-uCE
+CE_BQ24
 Text Notes 850  5550 0    50   ~ 0
 * 1 ON  , 2 OFF: Stand Alone\n* 1 OFF , 2 ON : u Controlled
@@
 Text Label 1000 3750 3    50   ~ 0
 VREF
-Text Label 5900 6050 3    50   ~ 0
+Text Label 5700 6050 3    50   ~ 0
 VREF
 Wire Wire Line
-	5900 6050 5900 6300
+	5700 6050 5700 6300
 $Comp
 L Connector:TestPoint TP3
@@
 L Connector:TestPoint TP5
 U 1 1 6155EE9E
-P 5150 6250
-F 0 "TP5" H 5100 6600 50  0000 L CNN
-F 1 "VCC" H 5100 6500 50  0000 L CNN
-F 2 "TestPoint:KEYSTONE_5016" H 5350 6250 50  0001 C CNN
-F 3 "~" H 5350 6250 50  0001 C CNN
-	1    5150 6250
-	1    0    0    -1
-$EndComp
-Text Label 5150 6250 3    50   ~ 0
+P 4850 6250
+F 0 "TP5" H 4800 6600 50  0000 L CNN
+F 1 "VCC" H 4800 6500 50  0000 L CNN
+F 2 "TestPoint:KEYSTONE_5016" H 5050 6250 50  0001 C CNN
+F 3 "~" H 5050 6250 50  0001 C CNN
+	1    4850 6250
+	1    0    0    -1
+$EndComp
+Text Label 4850 6250 3    50   ~ 0
 VCC
 $Comp
@@
 Text Label 1500 7600 1    50   ~ 0
 GND_BAT
-Text Label 5150 7500 1    50   ~ 0
+Text Label 4850 7500 1    50   ~ 0
 GNDA
 Text Label 8400 5600 3    50   ~ 0
@@
 GND_BAT
 Wire Notes Line
-	2050 5600 650  5600
+	2050 5600 550  5600
 Text HLabel 1850 7550 2    50   Output ~ 0
 GNDA

Commit message: Adds final pcb
Parts:
- NT1: footprint NetTie:NetTie-3_SMD_Pad0.5mm -> NetTie:NetTie-2_SMD_Pad2.0mm
- U3: footprint Package_DFN_QFN:VQFN-24-1EP_4x4mm_P0.5mm_EP2.45x2.45mm -> Package_DFN_QFN:VQFN-24-1EP_4x4mm_P0.5mm_EP2.45x2.45mm_ThermalVias
Changed lines of the file:
@@
 $Descr A4 11693 8268
 encoding utf-8
-Sheet 5 8
+Sheet 5 9
 Title ""
 Date ""
@@
 F 0 "U3" H 3400 6900 60  0000 L CNN
 F 1 "BQ24618RGET" H 3250 6800 60  0000 L CNN
-F 2 "Package_DFN_QFN:VQFN-24-1EP_4x4mm_P0.5mm_EP2.45x2.45mm" H 3700 6790 60  0001 C CNN
+F 2 "Package_DFN_QFN:VQFN-24-1EP_4x4mm_P0.5mm_EP2.45x2.45mm_ThermalVias" H 3700 6790 60  0001 C CNN
 F 3 "https://ar.mouser.com/ProductDetail/595-BQ24618RGET/" H 2700 6550 60  0001 C CNN
 	2    2700 6550
@@
 F 0 "NT1" H 1650 7381 50  0000 C CNN
 F 1 "GND-TIE" H 1650 7290 50  0000 C CNN
-F 2 "NetTie:NetTie-3_SMD_Pad0.5mm" H 1650 7200 50  0001 C CNN
+F 2 "NetTie:NetTie-2_SMD_Pad2.0mm" H 1650 7200 50  0001 C CNN
 F 3 "~" H 1650 7200 50  0001 C CNN
 	1    1650 7200
@@
 F 0 "U3" H 5050 3837 60  0000 C CNN
 F 1 "BQ24618RGET" H 5050 3731 60  0000 C CNN
-F 2 "Package_DFN_QFN:VQFN-24-1EP_4x4mm_P0.5mm_EP2.45x2.45mm" H 5050 3690 60  0001 C CNN
+F 2 "Package_DFN_QFN:VQFN-24-1EP_4x4mm_P0.5mm_EP2.45x2.45mm_ThermalVias" H 5050 3690 60  0001 C CNN
 F 3 "https://ar.mouser.com/ProductDetail/595-BQ24618RGET/" H 4050 3450 60  0001 C CNN
 	1    4050 3450

Commit message: Mirrors in x axis J3
Other:
- moved on the sheet: J3
Changed lines of the file:
@@
 	1    0    0    -1
 $EndComp
-Wire Wire Line
-	1950 1300 1950 1700
-Wire Wire Line
-	1950 1800 1950 2350
 $Comp
 L Connector_Generic:Conn_01x02 J3
 U 1 1 5FF53E53
-P 1750 1800
-F 0 "J3" H 1830 1700 50  0000 L CNN
-F 1 "Vcc In" H 1830 1791 50  0000 L CNN
-F 2 "Connector_Molex:Molex_KK-396_A-41791-0002_1x02_P3.96mm_Vertical" H 1750 1800 50  0001 C CNN
-F 3 "https://www.mouser.com/ProductDetail/571-1744429-2/" H 1750 1800 50  0001 C CNN
-	1    1750 1800
-	-1   0    0    1
+P 1750 1750
+F 0 "J3" H 1830 1650 50  0000 L CNN
+F 1 "Vcc In" H 1830 1741 50  0000 L CNN
+F 2 "Connector_Molex:Molex_KK-396_A-41791-0002_1x02_P3.96mm_Vertical" H 1750 1750 50  0001 C CNN
+F 3 "https://www.mouser.com/ProductDetail/571-1744429-2/" H 1750 1750 50  0001 C CNN
+	1    1750 1750
+	-1   0    0    -1
 $EndComp
 Wire Wire Line
@@
 	0    1    -1   0
 $EndComp
+Wire Wire Line
+	1950 1300 1950 1750
+Wire Wire Line
+	1950 1850 1950 2350
 $EndSCHEMATC
