File: bat_charger.sch (KiCad schematic (older format))
At the start: 59 parts, among them J3 Vcc In, J4 CH_TS, Q10 FDD86580-F085, Q7 DMP4051LK3, Q8 DMP4051LK3, Q9 FDD86580-F085, SW1 Reset, SW2 Select CE, U3 BQ24618RGET

Commit message: who knows
Other:
- note added: "Input"
- note removed: "Imput"
Changed lines of the file:
@@
 	5850 500  5850 2800
 Text Notes 5400 650  0    59   ~ 12
-Imput
+Input
 Text Notes 10800 650  0    59   ~ 12
 Output
