File: equalizer_bq76.sch (KiCad schematic (older format))
At the start: 16 parts, among them J2 Conn_01x07_Female, U2 BQ76PL536APAPR

Commit message: Edited sch page settings & printed schematic pdf
Parts:
- U2: symbol Battery_Management:BQ76PL536APAPR -> bms_hardware-rescue:BQ76PL536APAPR-Battery_Management
Changed lines of the file:
@@
 encoding utf-8
 Sheet 3 9
-Title ""
+Title "Battery Managment System (MBS)"
 Date ""
 Rev "A"
-Comp ""
+Comp "Ceccarelli Federico, Moya Martin,  Santos Lucio"
 Comment1 ""
-Comment2 ""
-Comment3 ""
-Comment4 ""
+Comment2 "Universidad Nacional de Rosario (UNR)"
+Comment3 "Facultad de Ciencias Exactas, Ingeniería y Agrimensura"
+Comment4 "Proyecto Final - Ingeniería Electrónica"
 $EndDescr
 Wire Wire Line
@@
 	4950 4150 4950 4250
 $Comp
-L Battery_Management:BQ76PL536APAPR U2
+L bms_hardware-rescue:BQ76PL536APAPR-Battery_Management U2
 U 1 1 603E20E4
 P 4050 3750
